File: RF/RF/Balun.kicad_sch (KiCad schematic)
At the start: 1 part, among them U301 0433BM15A0001

Commit message: added external memory
Connections:
- net Unbalanced_RF renamed UNBALANCED_RF
Other:
- moved on the sheet: U301
Changed lines of the file:
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@@
     (company "By: Atharva Kulkarni")
   )
-  (wire (pts (xy 142.24 74.676) (xy 149.86 74.676))
+  (wire (pts (xy 150.622 92.71) (xy 158.242 92.71))
     (stroke (width 0) (type default))
   )
-  (wire (pts (xy 142.24 76.454) (xy 142.24 74.676))
+  (wire (pts (xy 150.622 94.488) (xy 150.622 92.71))
     (stroke (width 0) (type default))
   )
-  (wire (pts (xy 131.572 78.994) (xy 134.62 78.994))
+  (wire (pts (xy 139.954 97.028) (xy 143.002 97.028))
     (stroke (width 0) (type default))
   )
-  (wire (pts (xy 149.86 74.676) (xy 149.86 79.756))
+  (wire (pts (xy 158.242 92.71) (xy 158.242 97.79))
     (stroke (width 0) (type default))
   )
-  (wire (pts (xy 144.78 89.154) (xy 146.812 89.154))
+  (wire (pts (xy 153.162 107.188) (xy 155.194 107.188))
     (stroke (width 0) (type default))
   )
-  (wire (pts (xy 132.334 89.154) (xy 134.62 89.154))
+  (wire (pts (xy 140.716 107.188) (xy 143.002 107.188))
     (stroke (width 0) (type default))
   )
-  (hierarchical_label "Unbalanced_RF" (shape output) (at 146.812 89.154 0) (fields_autoplaced)
+  (hierarchical_label "UNBALANCED_RF" (shape bidirectional) (at 155.194 107.188 0) (fields_autoplaced)
     (effects (font (size 1.27 1.27)) (justify left))
   )
-  (hierarchical_label "CC_RF_N" (shape input) (at 132.334 89.154 180) (fields_autoplaced)
+  (hierarchical_label "CC_RF_N" (shape input) (at 140.716 107.188 180) (fields_autoplaced)
     (effects (font (size 1.27 1.27)) (justify right))
   )
-  (hierarchical_label "CC_RF_P" (shape input) (at 131.572 78.994 180) (fields_autoplaced)
+  (hierarchical_label "CC_RF_P" (shape input) (at 139.954 97.028 180) (fields_autoplaced)
     (effects (font (size 1.27 1.27)) (justify right))
   )
-  (symbol (lib_id "Transformer:0433BM15A0001") (at 139.7 84.074 180) (unit 1)
+  (symbol (lib_id "Transformer:0433BM15A0001") (at 148.082 102.108 180) (unit 1)
     (in_bom yes) (on_board yes) (dnp no)
-    (property "Reference" "U301" (at 139.446 93.726 0)
+    (property "Reference" "U301" (at 147.828 111.76 0)
       (effects (font (size 1.27 1.27)))
     )
-    (property "Value" "0433BM15A0001" (at 139.7 91.694 0)
+    (property "Value" "0433BM15A0001" (at 148.082 109.728 0)
       (effects (font (size 1.27 1.27)))
     )
-    (property "Footprint" "RF_Converter:Balun_Johanson_0896BM15A0001" (at 139.7 76.454 0)
+    (property "Footprint" "RF_Converter:Balun_Johanson_0896BM15A0001" (at 148.082 94.488 0)
       (effects (font (size 1.27 1.27)) hide)
     )
-    (property "Datasheet" "https://www.johansontechnology.com/datasheets/0433BM15A0001/0433BM15A0001.pdf" (at 139.7 91.694 0)
+    (property "Datasheet" "https://www.johansontechnology.com/datasheets/0433BM15A0001/0433BM15A0001.pdf" (at 148.082 109.728 0)
       (effects (font (size 1.27 1.27)) hide)
     )
@@
     )
   )
-  (symbol (lib_id "power:GND") (at 149.86 79.756 0) (unit 1)
+  (symbol (lib_id "power:GND") (at 158.242 97.79 0) (unit 1)
     (in_bom yes) (on_board yes) (dnp no) (fields_autoplaced)
-    (property "Reference" "#PWR0301" (at 149.86 86.106 0)
+    (property "Reference" "#PWR0301" (at 158.242 104.14 0)
       (effects (font (size 1.27 1.27)) hide)
     )
-    (property "Value" "GND" (at 149.86 83.8915 0)
+    (property "Value" "GND" (at 158.242 101.9255 0)
       (effects (font (size 1.27 1.27)))
     )
-    (property "Footprint" "" (at 149.86 79.756 0)
+    (property "Footprint" "" (at 158.242 97.79 0)
       (effects (font (size 1.27 1.27)) hide)
     )
-    (property "Datasheet" "" (at 149.86 79.756 0)
+    (property "Datasheet" "" (at 158.242 97.79 0)
       (effects (font (size 1.27 1.27)) hide)
     )
