File: RF/RF/RF_front_end.kicad_sch (KiCad schematic)
At the start: 0 parts

Commit message: added external memory
Parts:
- added C501, C505, C506, C508: 0.1uF, Capacitor_SMD:C_0603_1608Metric_Pad1.08x0.95mm_HandSolder, symbol Device:C
- added C502, C503: 47uF, Capacitor_SMD:C_0603_1608Metric_Pad1.08x0.95mm_HandSolder, symbol Device:C
- added C504: 4.7uF, Capacitor_SMD:C_0603_1608Metric_Pad1.08x0.95mm_HandSolder, symbol Device:C
- added C507: 1uF, Capacitor_SMD:C_0603_1608Metric_Pad1.08x0.95mm_HandSolder, symbol Device:C
- added FB501: Z = 1k @ 100M, Inductor_SMD:L_0603_1608Metric_Pad1.05x0.95mm_HandSolder, symbol Device:FerriteBead
- added IC501: RFFM6406SR, SamacSys_Parts:RFFM6403, symbol SamacSys_Parts:RFFM6403
- added R501: 3.09k 1%, Resistor_SMD:R_0603_1608Metric_Pad0.98x0.95mm_HandSolder, symbol Device:R
- added R502: 6.65k 1%, Resistor_SMD:R_0603_1608Metric_Pad0.98x0.95mm_HandSolder, symbol Device:R
- added R503: 0R, Resistor_SMD:R_0603_1608Metric_Pad0.98x0.95mm_HandSolder, symbol Device:R
- added R504, R505: 1k, Resistor_SMD:R_0603_1608Metric_Pad0.98x0.95mm_HandSolder, symbol Device:R
Connections:
- new net: C502.1, C503.1, C504.1, C505.1, C506.1, C507.1, C508.1, IC501.17 (VCC_RX), IC501.23 (VDD), IC501.24 (VCC_TX1), IC501.26 (VCC_TX2), R503.1, R504.2
- new net: C501.1, FB501.1, R501.1
- new net +3.3V: FB501.2, R503.2
- new net ANTENNA: IC501.7 (ANT)
- new net GND: C501.2, C502.2, C503.2, C504.2, C505.2, C506.2, C507.2, C508.2, IC501.1 (GND_1), IC501.11 (GND_5), IC501.12 (GND_6), IC501.15 (GND_7), IC501.19 (GND_8), IC501.21 (GND_9), IC501.22 (GND_10), IC501.27 (GND_11), IC501.28 (GND_12), IC501.29 (EP), IC501.6 (GND_2), IC501.8 (GND_3), IC501.9 (GND_4), R502.2, R505.1
- new net LST_TX_MODE: IC501.2 (TR)
- new net PA_VAPC: IC501.5 (VAPC), R501.2, R502.1
- new net RF_BYP: IC501.4 (BYP), R505.2
- new net RF_EN: IC501.3 (EN), R504.1
- new net RX: IC501.18 (RX)
- new net SAW1: IC501.10 (SAW1)
- new net SAW2: IC501.13 (SAW2)
- new net TX: IC501.20 (TX)
- no-connect marks 0 -> 3
Other:
- note added: "Nominal VAPC = 2.25V @ 60 uA"

Commit message: RF: Push for schematic capture review version 1.0
Other:
- note added: "Look at pg 4 of Datasheet for control logic truth table"
Changed lines of the file:
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@@
     (stroke (width 0) (type default))
+  )
+  (text "Look at pg 4 of Datasheet for control logic truth table"
+    (at 56.896 61.976 0)
+    (effects (font (size 1.27 1.27)) (justify left bottom))
   )
   (text "Nominal VAPC = \n2.25V @ 60 uA" (at 121.412 46.228 0)
