File: RF/RF/RF_switch.kicad_sch (KiCad schematic)
At the start: 1 part, among them IC401 PE4250MLI-Z

Commit message: added external memory
Parts:
- added C401: 0.1uF, Capacitor_SMD:C_0603_1608Metric_Pad1.08x0.95mm_HandSolder, symbol Device:C
- added FB401: Z = 1k @ 100M, Inductor_SMD:L_0603_1608Metric_Pad1.05x0.95mm_HandSolder, symbol Device:FerriteBead
- added R401: DNP, Resistor_SMD:R_0603_1608Metric_Pad0.98x0.95mm_HandSolder, symbol Device:R
- added R402, R403: 0R, Resistor_SMD:R_0603_1608Metric_Pad0.98x0.95mm_HandSolder, symbol Device:R
- IC401: footprint SOP65P488X107-8N -> SamacSys_Parts:SOP65P488X107-8N
Connections:
- net at IC401.1 (V2): now also C401.1, FB401.2
- net at IC401.2 (V1): now also R401.2, R402.2
- net UNBALANCED_RF: now reaches IC401.3 (RFC)
- net GND: now reaches IC401.4 (N/C_OR_GND)
- net GND: now also IC401.6 (GND_1), IC401.7 (GND_2), C401.2
- net TX: now reaches IC401.5 (RF1)
- net RX: now reaches IC401.8 (RF2)
- new net: FB401.1, R403.1
- new net +3.3V: R401.1, R403.2
- new net ~{LST_RX_MODE}: R402.1
Other:
- note added: "Pulled to 3V3 via 10k pull up on CC110 schematic"
- note added: "V1 -> TX V2 -> RX"

Commit message: RF: Push for schematic capture review version 1.0
Other:
- note added: "(Pin 1 (V2) = VDD and Pin 2 (V1) = High) => RFC to RF1 (Pin 1 (V2) = VDD and Pin 2 (V1) = Low) => RFC to RF2 Pg 3 of datasheet"
- note removed: "V1 -> TX V2 -> RX"
Changed lines of the file:
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@@
     (effects (font (size 1.27 1.27)) (justify left bottom))
   )
-  (text "V1 -> TX\nV2 -> RX" (at 148.336 69.596 0)
+  (text "(Pin 1 (V2) = VDD and Pin 2 (V1) = High) => RFC to RF1\n(Pin 1 (V2) = VDD and Pin 2 (V1) = Low) => RFC to RF2\nPg 3 of datasheet"
+    (at 138.43 67.564 0)
     (effects (font (size 1.27 1.27)) (justify left bottom))
   )
