File: RF/RF/memory.kicad_sch (KiCad schematic)
At the start: 6 parts, among them IC701 23K256-I_SN, IC702 SST25VF512A-33-4C-SAE

Commit message: RF: Push for schematic capture review version 1.0
Connections:
- net ~{FRAM_CS} renamed ~{FLASH_CS}
Changed lines of the file:
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@@
     (stroke (width 0) (type default))
   )
-  (rectangle (start 51.816 62.992) (end 117.856 101.092)
-    (stroke (width 0) (type default))
+  (rectangle (start 51.816 61.722) (end 117.856 101.092)
+    (stroke (width 0.5) (type default))
     (fill (type none))
   )
   (rectangle (start 161.29 57.912) (end 256.54 101.6)
-    (stroke (width 0) (type default))
+    (stroke (width 0.5) (type default))
     (fill (type none))
   )
@@
     (effects (font (size 1.27 1.27)) (justify left))
   )
-  (hierarchical_label "~{FRAM_CS}" (shape input) (at 189.484 80.518 180) (fields_autoplaced)
+  (hierarchical_label "~{FLASH_CS}" (shape input) (at 189.484 80.518 180) (fields_autoplaced)
     (effects (font (size 1.27 1.27)) (justify right))
   )
