File: Flight Computer Board/FlightDeck_a/suck.kicad_sch (KiCad schematic)
At the start: 0 parts

Commit message: asdf
Parts:
- added J801: ESQ-110-13-G-D, SamacSys_Parts:ESQ-110-Y-X-D, symbol SamacSys_Parts:ESQ-110-13-G-D
Connections:
- new net +3.3V: J801.14, J801.18
- new net +5V: J801.10, J801.6
- new net CANH: J801.17
- new net CANL: J801.15
- new net GND: J801.12, J801.13, J801.16, J801.19, J801.20, J801.4, J801.8
- new net GPIO_1: J801.11
- new net GPIO_2: J801.9
- new net GPIO_3: J801.7
- new net GPIO_4: J801.5
- new net GPIO_5: J801.3
- new net GPIO_6: J801.1
- new net VBUS: J801.2
Other:
- note added: "MUMBAI STANDARD CONNECTOR"
