File: Flight Computer V2/Flight_Computer_V2/4-20maSignal_sch.kicad_sch (KiCad schematic)
At the start: 1 part

Commit message: more flgiht computer v2 updates
Other:
- note added: "4-20mA Sensor"
- moved on the sheet: R26
Changed lines of the file:
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@@
 (kicad_sch (version 20230121) (generator eeschema)
   (paper "A4")
-  (junction (at 93.98 57.15) (diameter 0) (color 0 0 0 0)
+  (junction (at 82.55 55.88) (diameter 0) (color 0 0 0 0)
   )
-  (wire (pts (xy 105.41 57.15) (xy 105.41 62.23))
+  (wire (pts (xy 93.98 55.88) (xy 93.98 60.96))
     (stroke (width 0) (type default))
   )
-  (wire (pts (xy 93.98 48.26) (xy 93.98 50.8))
+  (wire (pts (xy 82.55 49.53) (xy 82.55 52.07))
     (stroke (width 0) (type default))
   )
-  (wire (pts (xy 93.98 57.15) (xy 100.33 57.15))
+  (wire (pts (xy 82.55 55.88) (xy 88.9 55.88))
     (stroke (width 0) (type default))
   )
-  (wire (pts (xy 87.63 64.77) (xy 93.98 64.77))
+  (wire (pts (xy 76.2 63.5) (xy 82.55 63.5))
     (stroke (width 0) (type default))
   )
-  (wire (pts (xy 93.98 57.15) (xy 93.98 64.77))
+  (wire (pts (xy 82.55 55.88) (xy 82.55 63.5))
     (stroke (width 0) (type default))
   )
-  (wire (pts (xy 87.63 57.15) (xy 93.98 57.15))
+  (wire (pts (xy 76.2 55.88) (xy 82.55 55.88))
     (stroke (width 0) (type default))
   )
-  (wire (pts (xy 87.63 50.8) (xy 93.98 50.8))
+  (wire (pts (xy 76.2 52.07) (xy 82.55 52.07))
     (stroke (width 0) (type default))
+  )
+  (rectangle (start 60.96 49.53) (end 76.2 58.42)
+    (stroke (width 0) (type default))
+    (fill (type none))
+  )
+  (text "4-20mA Sensor\n" (at 60.96 49.53 0)
+    (effects (font (size 1.27 1.27)) (justify left bottom))
   )
   (text "Sense Resistor:\n220-245 for 5V ADC reference\n140-160 for 3.3V ADC reference"
@@
     (effects (font (size 1.27 1.27)) (justify left bottom))
   )
-  (hierarchical_label "420_OUT" (shape output) (at 87.63 57.15 180) (fields_autoplaced)
+  (hierarchical_label "420_OUT" (shape output) (at 76.2 55.88 180) (fields_autoplaced)
     (effects (font (size 1.27 1.27)) (justify right))
   )
-  (hierarchical_label "uC_IN" (shape input) (at 87.63 64.77 180) (fields_autoplaced)
+  (hierarchical_label "uC_IN" (shape input) (at 76.2 63.5 180) (fields_autoplaced)
     (effects (font (size 1.27 1.27)) (justify right))
   )
-  (hierarchical_label "420_IN" (shape input) (at 87.63 50.8 180) (fields_autoplaced)
+  (hierarchical_label "420_IN" (shape input) (at 76.2 52.07 180) (fields_autoplaced)
     (effects (font (size 1.27 1.27)) (justify right))
   )
-  (symbol (lib_id "Device:R_Small") (at 102.87 57.15 270) (unit 1)
+  (symbol (lib_id "Device:R_Small") (at 91.44 55.88 270) (unit 1)
     (in_bom yes) (on_board yes) (dnp no) (fields_autoplaced)
-    (property "Reference" "R26" (at 102.87 52.07 90)
+    (property "Reference" "R26" (at 91.44 50.8 90)
       (effects (font (size 1.27 1.27)))
     )
-    (property "Value" "150" (at 102.87 54.61 90)
+    (property "Value" "150" (at 91.44 53.34 90)
       (effects (font (size 1.27 1.27)))
     )
-    (property "Footprint" "" (at 102.87 57.15 0)
+    (property "Footprint" "" (at 91.44 55.88 0)
       (effects (font (size 1.27 1.27)) hide)
     )
-    (property "Datasheet" "~" (at 102.87 57.15 0)
+    (property "Datasheet" "~" (at 91.44 55.88 0)
       (effects (font (size 1.27 1.27)) hide)
     )
@@
     )
   )
-  (symbol (lib_id "power:VBUS") (at 93.98 48.26 0) (unit 1)
+  (symbol (lib_id "power:VBUS") (at 82.55 49.53 0) (unit 1)
     (in_bom yes) (on_board yes) (dnp no) (fields_autoplaced)
-    (property "Reference" "#PWR018" (at 93.98 52.07 0)
+    (property "Reference" "#PWR018" (at 82.55 53.34 0)
       (effects (font (size 1.27 1.27)) hide)
     )
-    (property "Value" "VBUS" (at 93.98 43.18 0)
+    (property "Value" "VBUS" (at 82.55 44.45 0)
       (effects (font (size 1.27 1.27)))
     )
-    (property "Footprint" "" (at 93.98 48.26 0)
+    (property "Footprint" "" (at 82.55 49.53 0)
       (effects (font (size 1.27 1.27)) hide)
     )
-    (property "Datasheet" "" (at 93.98 48.26 0)
+    (property "Datasheet" "" (at 82.55 49.53 0)
       (effects (font (size 1.27 1.27)) hide)
     )
@@
     )
   )
-  (symbol (lib_id "power:GND") (at 105.41 62.23 0) (unit 1)
+  (symbol (lib_id "power:GND") (at 93.98 60.96 0) (unit 1)
     (in_bom yes) (on_board yes) (dnp no)
-    (property "Reference" "#PWR03" (at 105.41 68.58 0)
+    (property "Reference" "#PWR03" (at 93.98 67.31 0)
       (effects (font (size 1.27 1.27)) hide)
     )
-    (property "Value" "GND" (at 105.41 66.04 0)
+    (property "Value" "GND" (at 93.98 64.77 0)
       (effects (font (size 1.27 1.27)))
     )
-    (property "Footprint" "" (at 105.41 62.23 0)
+    (property "Footprint" "" (at 93.98 60.96 0)
       (effects (font (size 1.27 1.27)) hide)
     )
-    (property "Datasheet" "" (at 105.41 62.23 0)
+    (property "Datasheet" "" (at 93.98 60.96 0)
       (effects (font (size 1.27 1.27)) hide)
     )

Commit message: finalized schematic, added datasheets, and pdf of schematic
Parts:
- added J5: Conn_01x02, symbol Connector_Generic:Conn_01x02
Connections:
- net VBUS: now also J5.2 (Pin_2)
- net 420_OUT renamed uC_IN
- net uC_IN: now also J5.1 (Pin_1)
Other:
- company: (none) -> By: Dylan Haussecker
- title: (none) -> Avionics Flight Computer
Changed lines of the file:
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@@
 (kicad_sch (version 20230121) (generator eeschema)
   (paper "A4")
+  (title_block
+    (title "Avionics Flight Computer")
+    (date "2023-09-04")
+    (rev "1.0")
+    (company "By: Dylan Haussecker")
+  )
   (junction (at 82.55 55.88) (diameter 0) (color 0 0 0 0)
   )
   (wire (pts (xy 93.98 55.88) (xy 93.98 60.96))
-    (stroke (width 0) (type default))
-  )
-  (wire (pts (xy 82.55 49.53) (xy 82.55 52.07))
     (stroke (width 0) (type default))
   )
@@
     (stroke (width 0) (type default))
   )
-  (wire (pts (xy 76.2 55.88) (xy 82.55 55.88))
+  (wire (pts (xy 64.77 55.88) (xy 82.55 55.88))
     (stroke (width 0) (type default))
   )
-  (wire (pts (xy 76.2 52.07) (xy 82.55 52.07))
+  (wire (pts (xy 82.55 49.53) (xy 82.55 53.34))
     (stroke (width 0) (type default))
   )
-  (rectangle (start 60.96 49.53) (end 76.2 58.42)
+  (wire (pts (xy 64.77 53.34) (xy 82.55 53.34))
+    (stroke (width 0) (type default))
+  )
+  (rectangle (start 53.34 43.18) (end 76.2 62.23)
     (stroke (width 0) (type default))
     (fill (type none))
   )
-  (text "4-20mA Sensor\n" (at 60.96 49.53 0)
+  (text "4-20mA Sensor\n" (at 53.34 43.18 0)
     (effects (font (size 1.27 1.27)) (justify left bottom))
   )
@@
     (effects (font (size 1.27 1.27)) (justify left bottom))
   )
-  (hierarchical_label "420_OUT" (shape output) (at 76.2 55.88 180) (fields_autoplaced)
-    (effects (font (size 1.27 1.27)) (justify right))
+  (label "420_IN" (at 66.04 53.34 0) (fields_autoplaced)
+    (effects (font (size 1.27 1.27)) (justify left bottom))
+  )
+  (label "420_OUT" (at 66.04 55.88 0) (fields_autoplaced)
+    (effects (font (size 1.27 1.27)) (justify left bottom))
   )
   (hierarchical_label "uC_IN" (shape input) (at 76.2 63.5 180) (fields_autoplaced)
     (effects (font (size 1.27 1.27)) (justify right))
   )
-  (hierarchical_label "420_IN" (shape input) (at 76.2 52.07 180) (fields_autoplaced)
-    (effects (font (size 1.27 1.27)) (justify right))
+  (symbol (lib_id "Connector_Generic:Conn_01x02") (at 59.69 55.88 180) (unit 1)
+    (in_bom yes) (on_board yes) (dnp no) (fields_autoplaced)
+    (property "Reference" "J5" (at 59.69 46.99 0)
+      (effects (font (size 1.27 1.27)))
+    )
+    (property "Value" "Conn_01x02" (at 59.69 49.53 0)
+      (effects (font (size 1.27 1.27)))
+    )
+    (property "Footprint" "" (at 59.69 55.88 0)
+      (effects (font (size 1.27 1.27)) hide)
+    )
+    (property "Datasheet" "~" (at 59.69 55.88 0)
+      (effects (font (size 1.27 1.27)) hide)
+    )
+    (pin "1")
+    (pin "2")
+    (instances
+      (project "Flight_Computer_V2"
+        (path "/39d7ebb3-b69d-4ae9-8f55-c9acfe77d345/cea5a790-cf79-44b4-a64b-a9c2141eca7e"
+          (reference "J5") (unit 1)
+        )
+        (path "/39d7ebb3-b69d-4ae9-8f55-c9acfe77d345/890b1d37-7c08-4080-9f9c-650c5e05f400"
+          (reference "J6") (unit 1)
+        )
+        (path "/39d7ebb3-b69d-4ae9-8f55-c9acfe77d345/9a670be6-a941-46a2-967f-f70de418761f"
+          (reference "J7") (unit 1)
+        )
+        (path "/39d7ebb3-b69d-4ae9-8f55-c9acfe77d345/e9e572b1-004c-4b07-9e39-8243b1fc8584"
+          (reference "J8") (unit 1)
+        )
+      )
+    )
   )
   (symbol (lib_id "Device:R_Small") (at 91.44 55.88 270) (unit 1)

Commit message: updated pcb
Parts:
- R26: footprint (none) -> Resistor_SMD:R_0402_1005Metric
Changed lines of the file:
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@@
       (effects (font (size 1.27 1.27)))
     )
-    (property "Footprint" "" (at 91.44 55.88 0)
+    (property "Footprint" "Resistor_SMD:R_0402_1005Metric" (at 91.44 55.88 0)
       (effects (font (size 1.27 1.27)) hide)
     )
