File: Flight Computer V2/Flight_Computer_V2/BMI088.kicad_sch (KiCad schematic)
At the start: 7 parts, among them IC5 BMI088

Commit message: finalized schematic, added datasheets, and pdf of schematic
Other:
- company: (none) -> By: Dylan Haussecker
- title: (none) -> Avionics Flight Computer
Changed lines of the file:
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@@
 (kicad_sch (version 20230121) (generator eeschema)
   (paper "A4")
+  (title_block
+    (title "Avionics Flight Computer")
+    (date "2023-09-04")
+    (rev "1.0")
+    (company "By: Dylan Haussecker")
+  )
   (junction (at 149.86 60.96) (diameter 0) (color 0 0 0 0)
   )

Commit message: updated pcb
Parts:
- C11, C19: footprint (none) -> Capacitor_SMD:C_0402_1005Metric
- IC5: footprint BMI088 -> LibraryLoader:BMI088
- JP3: footprint (none) -> Jumper:SolderJumper-2_P1.3mm_Open_Pad1.0x1.5mm
- TP3: footprint (none) -> TestPoint:TestPoint_Pad_D1.0mm
Changed lines of the file:
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@@
       (effects (font (size 1.27 1.27)))
     )
-    (property "Footprint" "" (at 156.21 60.96 0)
+    (property "Footprint" "Jumper:SolderJumper-2_P1.3mm_Open_Pad1.0x1.5mm" (at 156.21 60.96 0)
       (effects (font (size 1.27 1.27)) hide)
     )
@@
       (effects (font (size 1.27 1.27)) (justify left))
     )
-    (property "Footprint" "" (at 106.68 91.44 0)
+    (property "Footprint" "Capacitor_SMD:C_0402_1005Metric" (at 106.68 91.44 0)
       (effects (font (size 1.27 1.27)) hide)
     )
@@
       (effects (font (size 1.27 1.27)))
     )
-    (property "Footprint" "" (at 187.96 69.85 0)
+    (property "Footprint" "Jumper:SolderJumper-2_P1.3mm_Open_Pad1.0x1.5mm" (at 187.96 69.85 0)
       (effects (font (size 1.27 1.27)) hide)
     )
@@
       (effects (font (size 1.27 1.27)) (justify left) hide)
     )
-    (property "Footprint" "" (at 186.69 68.58 0)
+    (property "Footprint" "TestPoint:TestPoint_Pad_D1.0mm" (at 186.69 68.58 0)
       (effects (font (size 1.27 1.27)) hide)
     )
@@
       (effects (font (size 1.27 1.27)) (justify left))
     )
-    (property "Footprint" "" (at 179.07 86.36 0)
+    (property "Footprint" "Capacitor_SMD:C_0402_1005Metric" (at 179.07 86.36 0)
       (effects (font (size 1.27 1.27)) hide)
     )
@@
       (effects (font (size 1.27 1.27)) (justify right))
     )
-    (property "Footprint" "BMI088" (at 133.35 68.58 0)
+    (property "Footprint" "LibraryLoader:BMI088" (at 133.35 68.58 0)
       (effects (font (size 1.27 1.27)) (justify left) hide)
     )
@@
       (effects (font (size 1.27 1.27)) (justify left) hide)
     )
-    (property "Footprint" "" (at 154.94 59.69 0)
-      (effects (font (size 1.27 1.27)) hide)
-    )
+    (property "Footprint" "TestPoint:TestPoint_Pad_D1.0mm" (at 154.94 59.69 0)
+      (effects (font (size 1.27 1.27)) hide)
+    )
