File: Flight Computer V2/Flight_Computer_V2/MAX31855KASA+T.kicad_sch (KiCad schematic)
At the start: 11 parts, among them IC7 MAX31855KASA+T

Commit message: finalized schematic, added datasheets, and pdf of schematic
Parts:
- added J9: Conn_01x02, symbol Connector_Generic:Conn_01x02
Connections:
- net T+: now also J9.1 (Pin_1)
- net T-: now also J9.2 (Pin_2)
Other:
- company: (none) -> By: Dylan Haussecker
- title: (none) -> Avionics Flight Computer
Changed lines of the file:
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@@
 (kicad_sch (version 20230121) (generator eeschema)
   (paper "A4")
+  (title_block
+    (title "Avionics Flight Computer")
+    (date "2023-09-04")
+    (rev "1.0")
+    (company "By: Dylan Haussecker")
+  )
   (junction (at 116.84 95.25) (diameter 0) (color 0 0 0 0)
   )
@@
     (stroke (width 0) (type default))
   )
-  (wire (pts (xy 86.36 86.36) (xy 90.17 86.36))
+  (wire (pts (xy 80.01 86.36) (xy 90.17 86.36))
     (stroke (width 0) (type default))
   )
@@
     (stroke (width 0) (type default))
   )
-  (wire (pts (xy 86.36 81.28) (xy 90.17 81.28))
+  (wire (pts (xy 80.01 81.28) (xy 90.17 81.28))
     (stroke (width 0) (type default))
   )
@@
     (stroke (width 0) (type default))
   )
+  (wire (pts (xy 80.01 86.36) (xy 80.01 85.09))
+    (stroke (width 0) (type default))
+  )
   (wire (pts (xy 110.49 82.55) (xy 110.49 81.28))
     (stroke (width 0) (type default))
@@
     (stroke (width 0) (type default))
   )
+  (wire (pts (xy 80.01 81.28) (xy 80.01 82.55))
+    (stroke (width 0) (type default))
+  )
   (wire (pts (xy 110.49 81.28) (xy 101.6 81.28))
     (stroke (width 0) (type default))
+  )
+  (label "T+" (at 82.55 86.36 0) (fields_autoplaced)
+    (effects (font (size 1.27 1.27)) (justify left bottom))
+  )
+  (label "T-" (at 82.55 81.28 0) (fields_autoplaced)
+    (effects (font (size 1.27 1.27)) (justify left bottom))
   )
   (hierarchical_label "nCS" (shape output) (at 173.99 85.09 0) (fields_autoplaced)
@@
   (hierarchical_label "SCK" (shape output) (at 190.5 87.63 0) (fields_autoplaced)
     (effects (font (size 1.27 1.27)) (justify left))
-  )
-  (hierarchical_label "T+" (shape input) (at 86.36 86.36 180) (fields_autoplaced)
-    (effects (font (size 1.27 1.27)) (justify right))
-  )
-  (hierarchical_label "T-" (shape input) (at 86.36 81.28 180) (fields_autoplaced)
-    (effects (font (size 1.27 1.27)) (justify right))
   )
   (hierarchical_label "SO" (shape output) (at 158.75 82.55 0) (fields_autoplaced)
@@
         )
       )
+    )
+  )
+  (symbol (lib_id "Connector_Generic:Conn_01x02") (at 74.93 85.09 180) (unit 1)
+    (in_bom yes) (on_board yes) (dnp no) (fields_autoplaced)
+    (property "Reference" "J9" (at 74.93 76.2 0)
+      (effects (font (size 1.27 1.27)))
+    )
+    (property "Value" "Conn_01x02" (at 74.93 78.74 0)
+      (effects (font (size 1.27 1.27)))
+    )
+    (property "Footprint" "" (at 74.93 85.09 0)
+      (effects (font (size 1.27 1.27)) hide)
+    )
+    (property "Datasheet" "~" (at 74.93 85.09 0)
+      (effects (font (size 1.27 1.27)) hide)
+    )
+    (pin "1")
+    (pin "2")
+    (instances
+      (project "Flight_Computer_V2"
+        (path "/39d7ebb3-b69d-4ae9-8f55-c9acfe77d345/18b8eda5-ab3e-431c-bc45-74a94283215a"
+          (reference "J9") (unit 1)
+        )
+        (path "/39d7ebb3-b69d-4ae9-8f55-c9acfe77d345/f3b0a203-efef-48d6-a96f-d80f6600821a"
+          (reference "J10") (unit 1)
+        )
+        (path "/39d7ebb3-b69d-4ae9-8f55-c9acfe77d345/5078b2de-7be2-47cd-a266-5bbcaff0544f"
+          (reference "J11") (unit 1)
+        )
+      )

Commit message: updated pcb
Parts:
- C21: value 0.01p -> 1p; footprint (none) -> Capacitor_SMD:C_0402_1005Metric
- C22: footprint (none) -> Capacitor_SMD:C_0402_1005Metric
- FB1, FB4: footprint (none) -> Inductor_SMD:L_0805_2012Metric
- IC7: footprint SOIC127P600X175-8N -> LibraryLoader:SOIC127P600X175-8N
- JP1, JP2, JP3: footprint (none) -> Jumper:SolderJumper-2_P1.3mm_Open_Pad1.0x1.5mm
- TP1, TP2, TP3: footprint (none) -> TestPoint:TestPoint_Pad_D1.0mm
Changed lines of the file:
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@@
       (effects (font (size 1.27 1.27)) (justify left))
     )
-    (property "Value" "0.01p" (at 104.14 85.0963 0)
-      (effects (font (size 1.27 1.27)) (justify left))
-    )
-    (property "Footprint" "" (at 101.6 83.82 0)
+    (property "Value" "1p" (at 104.14 85.0963 0)
+      (effects (font (size 1.27 1.27)) (justify left))
+    )
+    (property "Footprint" "Capacitor_SMD:C_0402_1005Metric" (at 101.6 83.82 0)
       (effects (font (size 1.27 1.27)) hide)
     )
@@
       (effects (font (size 1.27 1.27)) hide)
     )
-    (property "Footprint" "" (at 92.71 88.138 90)
+    (property "Footprint" "Inductor_SMD:L_0805_2012Metric" (at 92.71 88.138 90)
       (effects (font (size 1.27 1.27)) hide)
     )
@@
       (effects (font (size 1.27 1.27)))
     )
-    (property "Footprint" "" (at 186.69 87.63 0)
+    (property "Footprint" "Jumper:SolderJumper-2_P1.3mm_Open_Pad1.0x1.5mm" (at 186.69 87.63 0)
       (effects (font (size 1.27 1.27)) hide)
     )
@@
       (effects (font (size 1.27 1.27)))
     )
-    (property "Footprint" "" (at 170.18 85.09 0)
+    (property "Footprint" "Jumper:SolderJumper-2_P1.3mm_Open_Pad1.0x1.5mm" (at 170.18 85.09 0)
       (effects (font (size 1.27 1.27)) hide)
     )
@@
       (effects (font (size 1.27 1.27)) hide)
     )
-    (property "Footprint" "" (at 92.71 83.058 90)
+    (property "Footprint" "Inductor_SMD:L_0805_2012Metric" (at 92.71 83.058 90)
       (effects (font (size 1.27 1.27)) hide)
     )
@@
       (effects (font (size 1.27 1.27)) (justify left) hide)
     )
-    (property "Footprint" "" (at 170.18 83.82 0)
+    (property "Footprint" "TestPoint:TestPoint_Pad_D1.0mm" (at 170.18 83.82 0)
       (effects (font (size 1.27 1.27)) hide)
     )
@@
       (effects (font (size 1.27 1.27)) (justify left) hide)
     )
-    (property "Footprint" "" (at 154.94 81.28 0)
+    (property "Footprint" "TestPoint:TestPoint_Pad_D1.0mm" (at 154.94 81.28 0)
       (effects (font (size 1.27 1.27)) hide)
     )
@@
       (effects (font (size 1.27 1.27)) (justify left) hide)
     )
-    (property "Footprint" "" (at 186.69 86.36 0)
+    (property "Footprint" "TestPoint:TestPoint_Pad_D1.0mm" (at 186.69 86.36 0)
       (effects (font (size 1.27 1.27)) hide)
     )
@@
       (effects (font (size 1.27 1.27)))
     )
-    (property "Footprint" "SOIC127P600X175-8N" (at 143.51 77.47 0)
+    (property "Footprint" "LibraryLoader:SOIC127P600X175-8N" (at 143.51 77.47 0)
       (effects (font (size 1.27 1.27)) (justify left) hide)
     )
@@
       (effects (font (size 1.27 1.27)) (justify left))
     )
-    (property "Footprint" "" (at 116.84 97.79 0)
+    (property "Footprint" "Capacitor_SMD:C_0402_1005Metric" (at 116.84 97.79 0)
       (effects (font (size 1.27 1.27)) hide)
     )
@@
       (effects (font (size 1.27 1.27)))
     )
-    (property "Footprint" "" (at 154.94 82.55 0)
-      (effects (font (size 1.27 1.27)) hide)
-    )
+    (property "Footprint" "Jumper:SolderJumper-2_P1.3mm_Open_Pad1.0x1.5mm" (at 154.94 82.55 0)
+      (effects (font (size 1.27 1.27)) hide)
+    )
