File: Flight Computer V2/Flight_Computer_V2/State_Indication.kicad_sch (KiCad schematic)
At the start: 7 parts

Commit message: finalized schematic, added datasheets, and pdf of schematic
Other:
- company: (none) -> By: Dylan Haussecker
- title: (none) -> Avionics Flight Computer
Changed lines of the file:
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@@
 (kicad_sch (version 20230121) (generator eeschema)
   (paper "A4")
+  (title_block
+    (title "Avionics Flight Computer")
+    (date "2023-09-04")
+    (rev "1.0")
+    (company "By: Dylan Haussecker")
+  )
   (junction (at 153.67 83.82) (diameter 0) (color 0 0 0 0)
   )

Commit message: updated pcb
Parts:
- BZ1: footprint (none) -> Buzzer_Beeper:Buzzer_Murata_PKMCS0909E
- D4, D5, D6: footprint (none) -> LED_SMD:LED_0603_1608Metric
- R10, R11, R12: value 120 -> 500; footprint (none) -> Resistor_SMD:R_0603_1608Metric
Changed lines of the file:
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@@
       (effects (font (size 1.27 1.27)) (justify left))
     )
-    (property "Footprint" "" (at 89.535 64.77 90)
+    (property "Footprint" "Buzzer_Beeper:Buzzer_Murata_PKMCS0909E" (at 89.535 64.77 90)
       (effects (font (size 1.27 1.27)) hide)
     )
@@
       (effects (font (size 1.27 1.27)))
     )
-    (property "Value" "120" (at 137.16 60.96 90)
+    (property "Value" "500" (at 137.16 60.96 90)
       (effects (font (size 1.27 1.27)))
     )
-    (property "Footprint" "" (at 137.16 63.5 0)
+    (property "Footprint" "Resistor_SMD:R_0603_1608Metric" (at 137.16 63.5 0)
       (effects (font (size 1.27 1.27)) hide)
     )
@@
       (effects (font (size 1.27 1.27)))
     )
-    (property "Footprint" "" (at 144.78 83.82 90)
+    (property "Footprint" "LED_SMD:LED_0603_1608Metric" (at 144.78 83.82 90)
       (effects (font (size 1.27 1.27)) hide)
     )
@@
       (effects (font (size 1.27 1.27)))
     )
-    (property "Value" "120" (at 137.16 71.12 90)
+    (property "Value" "500" (at 137.16 71.12 90)
       (effects (font (size 1.27 1.27)))
     )
-    (property "Footprint" "" (at 137.16 73.66 0)
+    (property "Footprint" "Resistor_SMD:R_0603_1608Metric" (at 137.16 73.66 0)
       (effects (font (size 1.27 1.27)) hide)
     )
@@
       (effects (font (size 1.27 1.27)))
     )
-    (property "Footprint" "" (at 144.78 63.5 90)
+    (property "Footprint" "LED_SMD:LED_0603_1608Metric" (at 144.78 63.5 90)
       (effects (font (size 1.27 1.27)) hide)
     )
@@
       (effects (font (size 1.27 1.27)))
     )
-    (property "Footprint" "" (at 144.78 73.66 90)
+    (property "Footprint" "LED_SMD:LED_0603_1608Metric" (at 144.78 73.66 90)
       (effects (font (size 1.27 1.27)) hide)
     )
@@
       (effects (font (size 1.27 1.27)))
     )
-    (property "Value" "120" (at 137.16 81.28 90)
+    (property "Value" "500" (at 137.16 81.28 90)
       (effects (font (size 1.27 1.27)))
     )
-    (property "Footprint" "" (at 137.16 83.82 0)
+    (property "Footprint" "Resistor_SMD:R_0603_1608Metric" (at 137.16 83.82 0)
       (effects (font (size 1.27 1.27)) hide)
     )
